File: test/test.kicad_pcb (KiCad board)
At the start: 2 copper layers, 12.7 x 17.8 mm, 2 parts, among them J1 Conn_01x04, Y1 8MHz

Commit message: update
Routing:
- net Net-(J1-Pad1): track 0.00 -> 16.5 mm, vias 0 -> 2
- net Net-(J1-Pad3): track 0.00 -> 14.0 mm, vias 0 -> 2
- net Net-(J1-Pad2): track 0.00 -> 11.4 mm
Changed lines of the file:
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@@
   (general
     (links 3)
-    (no_connects 3)
-    (area 0 0 0 0)
+    (no_connects 0)
+    (area 142.164999 97.714999 155.015001 115.645001)
     (thickness 1.6)
     (drawings 4)
-    (tracks 0)
+    (tracks 13)
     (zones 0)
     (modules 2)
@@
     (pad_to_mask_clearance 0.2)
     (aux_axis_origin 0 0)
-    (visible_elements FFFFFF7F)
+    (visible_elements 7FFFFFFF)
     (pcbplotparams
       (layerselection 0x00030_80000001)
@@
   (module Connector_PinHeader_2.54mm:PinHeader_1x04_P2.54mm_Horizontal (layer F.Cu)
     (at 148.59 111.76)
-    (fp_text reference J1 (at -2.54 5.08) (layer F.SilkS)
+    (fp_text reference J1 (at -3.81 -2.54) (layer F.SilkS)
       (effects (font (size 1 1) (thickness 0.15)))
     )
@@
   (gr_line (start 154.94 97.79) (end 154.94 115.57) (angle 90) (layer Edge.Cuts) (width 0.15))
   (gr_line (start 142.24 97.79) (end 154.94 97.79) (angle 90) (layer Edge.Cuts) (width 0.15))
+  (segment (start 151.13 101.6) (end 151.13 106.68) (width 0.25) (layer B.Cu) (net 2) (status 400000))
+  (segment (start 147.32 106.68) (end 147.32 111.76) (width 0.25) (layer B.Cu) (net 2) (status 800000))
+  (via (at 147.32 106.68) (size 0.6) (drill 0.4) (layers F.Cu B.Cu) (net 2))
+  (segment (start 151.13 106.68) (end 147.32 106.68) (width 0.25) (layer F.Cu) (net 2))
+  (via (at 151.13 106.68) (size 0.6) (drill 0.4) (layers F.Cu B.Cu) (net 2))
+  (segment (start 148.59 101.6) (end 148.59 105.41) (width 0.25) (layer B.Cu) (net 3) (status 400000))
+  (segment (start 149.86 105.41) (end 149.86 111.76) (width 0.25) (layer B.Cu) (net 3) (status 800000))
+  (segment (start 148.59 105.41) (end 149.86 105.41) (width 0.25) (layer B.Cu) (net 3))
+  (segment (start 146.05 101.6) (end 146.05 107.95) (width 0.25) (layer B.Cu) (net 4) (status 400000))
+  (segment (start 152.4 107.95) (end 152.4 111.76) (width 0.25) (layer B.Cu) (net 4) (status 800000))
+  (via (at 152.4 107.95) (size 0.6) (drill 0.4) (layers F.Cu B.Cu) (net 4))
+  (segment (start 146.05 107.95) (end 152.4 107.95) (width 0.25) (layer F.Cu) (net 4))
+  (via (at 146.05 107.95) (size 0.6) (drill 0.4) (layers F.Cu B.Cu) (net 4))
 )
